File: SolenoidArray_Rev2.kicad_pcb (KiCad board)
At the start: 2 copper layers, 750.7 x 332.5 mm, 112 parts, among them J1 Conn_01x02, J10 Conn_01x02, J11 Conn_01x02, J12 Conn_01x02, J13 Conn_01x02, J14 Conn_01x02, J15 Conn_01x02, J16 Power Daisy Chain_input, J17 Power Daisy Chain_Output, J18 Arduino Pins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

Commit message: .
Parts:
- moved R16 8.22 mm to (380.1, 172.7), turned to 90 degrees
Routing:
- net Net-(J18-Pad16): track 233.3 -> 241.4 mm
Other:
- board text added: "MENO"
- board text added: "PIÙ e"
