File: SolenoidArray_Rev2.sch (KiCad schematic (older format))
At the start: 112 parts, among them J1 Conn_01x02, J10 Conn_01x02, J11 Conn_01x02, J12 Conn_01x02, J13 Conn_01x02, J14 Conn_01x02, J15 Conn_01x02, J16 Power Daisy Chain_input, J17 Power Daisy Chain_Output, J18 Arduino Pins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

Commit message: .
Other:
- moved on the sheet: C1, C2, D1, D10, D11, D12, D13, D14, D15, D16, D17, D18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
